Commit message: Use real Cycloidal R20 drive mesh at each joint in the sim
Converted Assy_Cycloid_R20_v0.STEP (ratio-20 cycloidal drive, 63.5mm sq x
57.4mm) to a recentered binary STL (axis=Z, base=z0, ~73k tris) via gmsh,
and swapped the placeholder joint cylinders in arm_trunk.urdf for this mesh
(one asset instanced 3x, scaled mm->m, oriented to each joint axis).
Per-part STLs in the package are print-oriented, so the STEP assembly is the
only source of true relative positions. Visual only; inertials unchanged.

Co-Authored-By: Claude Opus 4.8 <noreply@anthropic.com>

File: sim/arm_trunk.urdf (robot description, URDF)
Before this commit: robot cycloid_trunk, 5 links, 4 joints
Links:
- link forearm_link: geometry visual cylinder length=0.006 radius=0.022; visual cylinder length=0.060 radius=0.006
- link mast_link: geometry visual cylinder length=0.070 radius=0.023; visual mesh filename=cycloid_r20.stl scale=0.001 0.001 0.001
- link upper_arm_link: geometry visual cylinder length=0.210 radius=0.021; visual mesh filename=cycloid_r20.stl scale=0.001 0.001 0.001

Commit message: Mechanically faithful R20 joints: split drive, real motor, flat members
- Split the R20 STEP into FIXED half (motor plate + the real stepper, which
  is shell geometry in the STEP, + screws) and OUTPUT body (rotating ring
  wheels). Each joint straddles the revolute joint: motor mesh on the parent
  link, body mesh on the child -> the round output body rotates against the
  fixed motor like the real actuator.
- Drives centered on the joint so the two segments bolt to opposite ends and
  are offset ~36 mm; J2/J3 alternate side (+Y/-Y) so the arm zig-zags and
  segments clear. Round mounting plates match the round output face.
- Arm segments modeled as flat plate members. Real stepper now visible for
  clearance checks (note: STEP models it ~21 mm deep, shorter than a full
  NEMA17). J1 motor points down into the base pedestal.
- Removed the unused single-piece cycloid_r20.stl.

Co-Authored-By: Claude Opus 4.8 <noreply@anthropic.com>

File: sim/arm_trunk.urdf (robot description, URDF)
Before this commit: robot cycloid_trunk, 5 links, 4 joints
Links:
- link base_link: mass 0.60 -> 1.0; geometry visual cylinder length=0.055 radius=0.045; visual mesh filename=r20_motor.stl scale=0.001 0.001 0.001
- link forearm_link: mass 0.30 -> 0.4; geometry visual box size=0.044 0.010 0.006; visual box size=0.044 0.010 0.210
- link mast_link: mass 0.40 -> 0.6; geometry visual box size=0.055 0.012 0.060; visual cylinder length=0.005 radius=0.0315
- link upper_arm_link: mass 0.35 -> 0.5; geometry visual box size=0.050 0.010 0.210; visual cylinder length=0.005 radius=0.0315
Joints:
- joint j1_yaw: origin xyz=0 0 0.040 -> xyz=0 0 0.073
- joint tcp_fixed: origin xyz=0 0 0.276 -> xyz=0 -0.0184 0.276

Commit message: Extend to 5-DOF: add wrist-pitch + tool-roll on 20:1 Micro cycloidal
Chain: J1 yaw, J2 shoulder-pitch, J3 elbow-pitch (R20), J4 wrist-pitch and
J5 tool-roll (Sweep 20:1 Micro). Dropped the forearm-roll (avoids roll
redundancy; pitch-then-tool-roll wrist as discussed).
- micro20.stl: Micro 20:1 drive from its STEP (internal ladder discs dropped
  to keep it light, ~21k tris). Single mesh, mounted on the parent (fixed)
  side at each wrist joint; child link articulates.
- view.py: keyboard now covers all joints (Q/A W/S E/D R/F T/G, X=reset);
  loop/readout generalized to model.nu.
Reach ~0.49 m preserved; all 5 joints verified controllable in the viewer.

Co-Authored-By: Claude Opus 4.8 <noreply@anthropic.com>

File: sim/arm_trunk.urdf (robot description, URDF)
Before this commit: robot cycloid_trunk_r20, 5 links, 4 joints
Links:
- added link tool_link, mass 0.08; visual cylinder length=0.006 radius=0.020; visual cylinder length=0.060 radius=0.006
- added link wrist_link, mass 0.15; visual box size=0.035 0.010 0.050; visual cylinder length=0.004 radius=0.020
- link forearm_link: mass 0.4 -> 0.35; geometry visual box size=0.044 0.010 0.150; visual cylinder length=0.004 radius=0.020
Joints:
- added joint j4_wrist_pitch: type revolute, parent forearm_link, child wrist_link, origin xyz=0 -0.0184 0.162, axis 0 1 0, limit lower=-1.92 upper=1.92 effort=6 velocity=3.0
- added joint j5_tool_roll: type revolute, parent wrist_link, child tool_link, origin xyz=0 -0.0184 0.050, axis 0 0 1, limit lower=-3.1416 upper=3.1416 effort=4 velocity=3.0
- joint tcp_fixed: origin xyz=0 -0.0184 0.276 -> xyz=0 0 0.078; parent forearm_link -> tool_link

Commit message: assembly: use the MEASURED 188g full actuator (was ~320g estimate)
Real measured actuator weight (motor + cyclo) = 188 g. Fold it in, avoiding
double-counting: the actuator's printed housing/base are already in the section
mesh, so each section link = blade-only plastic + the 188g actuator (this
reduces exactly to blade_plastic + ACTUATOR). Link masses drop ~364g -> ~215g;
the arm is ~40% lighter than the estimate, unloading the shoulder.

Co-Authored-By: Claude Opus 4.8 <noreply@anthropic.com>

File: sim/arm_trunk.urdf (robot description, URDF)
Before this commit: robot micro_arm, 7 links, 6 joints
Links:
- link forearm_link: mass 0.3645 -> 0.2148
- link mast_link: mass 0.3400 -> 0.2080
- link upper_arm_link: mass 0.3645 -> 0.2148
- link wrist_link: mass 0.3200 -> 0.2080

Commit message: Calibrate to measured prototype: 75mm sections, pancake stepper, 1.32 N*m
Real measurements from the prototype:
- SEG=75mm (joint-to-joint), pancake stepper actuator (188g, light/weak).
- Joint torque cap = 1.32 N*m output (1.8kg on a scale at 75mm), where the
  OPEN-LOOP STEPPER misses steps -- the printed cyclo does NOT slip, so it's an
  electrical limit (tunable: more current / closed-loop), not mechanical.
- Set as the micro joints' effort + gravity.py TAU.

Sim finding at 75mm + 250g payload, dead-horizontal: shoulder needs 1.42 N*m
(~8% over the 1.32 cap -> drops steps); elbow 0.77, wrist 0.27 (both fine).

Co-Authored-By: Claude Opus 4.8 <noreply@anthropic.com>

File: sim/arm_trunk.urdf (robot description, URDF)
Before this commit: robot micro_arm, 7 links, 6 joints
Links:
- link forearm_link: mass 0.2148 -> 0.1984
- link upper_arm_link: mass 0.2148 -> 0.1984
Joints:
- joint j1_yaw: limit lower=-3.1416 upper=3.1416 effort=20 velocity=3.0 -> lower=-3.1416 upper=3.1416 effort=3.0 velocity=3.0
- joint j2_shoulder: limit lower=-1.9200 upper=1.9200 effort=18 velocity=3.0 -> lower=-1.9200 upper=1.9200 effort=1.32 velocity=3.0
- joint j3_elbow: limit lower=-2.6200 upper=2.6200 effort=15 velocity=3.0 -> lower=-2.6200 upper=2.6200 effort=1.32 velocity=3.0; origin xyz=0.1500 -0.0046 0.0000 -> xyz=0.0750 -0.0046 0.0000
- joint j4_wrist_pitch: limit lower=-1.9200 upper=1.9200 effort=6 velocity=3.0 -> lower=-1.9200 upper=1.9200 effort=1.32 velocity=3.0; origin xyz=0.1500 -0.0046 0.0000 -> xyz=0.0750 -0.0046 0.0000
- joint j5_tool_roll: limit lower=-3.1416 upper=3.1416 effort=4 velocity=3.0 -> lower=-3.1416 upper=3.1416 effort=1.32 velocity=3.0

Commit message: assembly: bigger shoulder motor (J2 at the base = free weight)
J2 sits at the base, so a heavier/stronger motor there loads only the slew, not
the arm (heavy-where-it-lifts). Per-joint actuator: NEMA17 at the shoulder
(ACTUATOR_SHOULDER=0.32kg, TORQUE_SHOULDER=3.0 N*m); keep the tiny pancake
(1.32 N*m) at J3-J5 where weight hangs. Shoulder now holds the 75mm arm + 250g
comfortably (1.42/3.0) and would hold up to ~150mm sections. (Caveat: the micro
cyclo is only confirmed to 1.32 N*m -- verify it transmits 3 before relying.)

Co-Authored-By: Claude Opus 4.8 <noreply@anthropic.com>

File: sim/arm_trunk.urdf (robot description, URDF)
Before this commit: robot micro_arm, 7 links, 6 joints
Links:
- link mast_link: mass 0.2080 -> 0.3400
Joints:
- joint j2_shoulder: limit lower=-1.9200 upper=1.9200 effort=1.32 velocity=3.0 -> lower=-1.9200 upper=1.9200 effort=3.0 velocity=3.0

Commit message: assembly: wire the right-angle bracket in as the base->shoulder section
mast_link is now the shoulder_bracket mesh (was a stand-in box); j2_shoulder
sits at the bracket's vertical-face bore. arm_assembly exports the bracket mesh
and the CAD preview includes it.

Co-Authored-By: Claude Opus 4.8 <noreply@anthropic.com>

File: sim/arm_trunk.urdf (robot description, URDF)
Before this commit: robot micro_arm, 7 links, 6 joints
Links:
- link mast_link: mass 0.3400 -> 0.3830; geometry visual mesh filename=shoulder_bracket.stl scale=0.001 0.001 0.001
Joints:
- joint j2_shoulder: origin xyz=0.0000 0.0000 0.0550 -> xyz=0.0000 -0.0270 0.0340

Commit message: assembly: wire the wrist box bracket in as the wrist section
wrist_link is now the wrist_bracket mesh (was a stand-in box), rotated off the
wrist-pitch output. arm_assembly exports it + supports mesh offset/rpy in the
URDF emitter; CAD preview includes it. The full arm now carries both real
90deg brackets (base + wrist).

Co-Authored-By: Claude Opus 4.8 <noreply@anthropic.com>

File: sim/arm_trunk.urdf (robot description, URDF)
Before this commit: robot micro_arm, 7 links, 6 joints
Links:
- link wrist_link: mass 0.2080 -> 0.2550; geometry visual mesh filename=wrist_bracket.stl scale=0.001 0.001 0.001

Commit message: assembly: wrist is the right-angle linkage (angle_drive), 5-DOF
Per the design: stay 5-DOF (no forearm-roll / double-90). The wrist section is now
the angle_drive right-angle linkage (cyclo body + NEMA plate) instead of the
slide-in box -- the wrist-pitch cyclo output carries the tool-roll motor at 90deg.
Swapped wrist_bracket -> angle_drive in the chain + mesh export; j5 re-placed at
the NEMA-plate face. (wrist_bracket.py is now unused.)

Co-Authored-By: Claude Opus 4.8 <noreply@anthropic.com>

File: sim/arm_trunk.urdf (robot description, URDF)
Before this commit: robot micro_arm, 7 links, 6 joints
Links:
- link wrist_link: mass 0.2550 -> 0.2180; geometry visual mesh filename=angle_drive.stl scale=0.001 0.001 0.001
Joints:
- joint j5_tool_roll: origin xyz=0.0500 0.0000 0.0000 -> xyz=0.0270 -0.0090 0.0000

Commit message: assembly: motor ladder (38/48/38/24) + 52mm forearm in the sim
Rework arm_assembly to match the real build's motor plan: per-joint torque caps
and actuator masses from the NEMA17 ladder (slew 38 / shoulder 48 / elbow 38 /
wrist 24), output torque anchored to the measured 24mm step-loss (1.32 N*m) and
scaled by holding torque. Two distinct section meshes: upper arm 75mm (carries
the 38mm elbow motor), forearm/last-pivot 52mm (carries the 24mm wrist motor).

Gravity hold @ horizontal: shoulder 1.28/5.5 N*m (4.3x), elbow 0.56/3.6 (6.5x),
wrist-pitch 0.20/1.32 (6.5x), slew/roll ~0 (their axes carry no gravity). The
ladder holds the 2.45kg arm + 0.25kg payload with margin everywhere.

(Geometry meshes for the cyclo_cage base + angle_mount wrist are still the older
cosmetic stand-ins; kinematics/dynamics now match the build.)

Co-Authored-By: Claude Opus 4.8 <noreply@anthropic.com>

File: sim/arm_trunk.urdf (robot description, URDF)
Before this commit: robot micro_arm, 7 links, 6 joints
Links:
- link forearm_link: mass 0.1984 -> 0.1933; geometry visual mesh filename=arm_fore.stl scale=0.001 0.001 0.001
- link mast_link: mass 0.3830 -> 0.4530
- link upper_arm_link: mass 0.1984 -> 0.3004; geometry visual mesh filename=arm_upper.stl scale=0.001 0.001 0.001
Joints:
- joint j1_yaw: limit lower=-3.1416 upper=3.1416 effort=3.0 velocity=3.0 -> lower=-3.1416 upper=3.1416 effort=3.6 velocity=3.0
- joint j2_shoulder: limit lower=-1.9200 upper=1.9200 effort=3.0 velocity=3.0 -> lower=-1.9200 upper=1.9200 effort=5.5 velocity=3.0
- joint j3_elbow: limit lower=-2.6200 upper=2.6200 effort=1.32 velocity=3.0 -> lower=-2.6200 upper=2.6200 effort=3.6 velocity=3.0
- joint j4_wrist_pitch: origin xyz=0.0750 -0.0046 0.0000 -> xyz=0.0520 -0.0046 0.0000

Commit message: assembly: render the real modular parts (cyclo_cage base + angle_mount wrist)
Swap the cosmetic stand-ins for the actual CAD: base_link is now the cyclo_cage
(slew drive, feet on the ground), and the wrist is angle_mount -- body_boss +
mount_plate combined into one wrist_assembly() solid that moves with J4. The sim
visual now matches the build (kinematics/dynamics already did). Wrist/tool fine
placement carried over from angle_drive and may want a small tune.

Co-Authored-By: Claude Opus 4.8 <noreply@anthropic.com>

File: sim/arm_trunk.urdf (robot description, URDF)
Before this commit: robot micro_arm, 7 links, 6 joints
Links:
- link base_link: mass 1.0000 -> 0.5000; geometry visual mesh filename=cyclo_cage.stl scale=0.001 0.001 0.001
- link wrist_link: geometry visual mesh filename=angle_wrist.stl scale=0.001 0.001 0.001

Commit message: Prune obsolete parts; keep only the current set
Remove the superseded parts and their artifacts: wrist_bracket, motor_cage,
angle_drive, shoulder_bracket. The current parts are arm_section, angle_mount
(body_boss + mount_plate = the 90deg connection used at BOTH the base slew and
the wrist), pivot_link, and cyclo_cage (base slew drive).

- cyclo_cage no longer imports motor_cage (inlined its leg/foot constants).
- arm_assembly drops shoulder_bracket; the base mast and the wrist both use the
  angle_mount solid (renamed wrist_assembly -> angle_mount_solid / angle_mount.stl).
- Makefile + CAD_NOTES references updated.

Co-Authored-By: Claude Opus 4.8 <noreply@anthropic.com>

File: sim/arm_trunk.urdf (robot description, URDF)
Before this commit: robot micro_arm, 7 links, 6 joints
Links:
- link mast_link: geometry visual mesh filename=angle_mount.stl scale=0.001 0.001 0.001
- link tool_link: geometry visual box size=0.022 0.05 0.026; visual box size=0.05 0.008 0.024
- link wrist_link: geometry visual mesh filename=angle_mount.stl scale=0.001 0.001 0.001
Joints:
- joint j1_yaw: origin xyz=0.0000 0.0000 0.0650 -> xyz=0.0000 0.0000 0.0470

Commit message: assembly: gripper tool + seat the upper arm on the base mount-plate boss
- tool_link is now a simple parallel-jaw gripper (palm + two fingers).
- base mast (angle_mount) rotated 90deg so the mount-plate bearing boss points
  along the shoulder axis (+Y); j2 origin moved onto the boss (z~42mm) so the
  upper arm's round body seats on it instead of floating.

Co-Authored-By: Claude Opus 4.8 <noreply@anthropic.com>

File: sim/arm_trunk.urdf (robot description, URDF)
Before this commit: robot micro_arm, 7 links, 6 joints
Joints:
- joint j2_shoulder: origin xyz=0.0000 -0.0270 0.0340 -> xyz=0.0000 0.0360 0.0420

Commit message: assembly: orient the wrist so the gripper points forward
Roll-flip the wrist angle_mount (rpy -pi/2) so the body still mates the forearm
but the mount-plate output (the perpendicular tool-roll axis) faces +X; move j5
onto that output so the gripper extends forward instead of pointing back.

Co-Authored-By: Claude Opus 4.8 <noreply@anthropic.com>

File: sim/arm_trunk.urdf (robot description, URDF)
Before this commit: robot micro_arm, 7 links, 6 joints
Joints:
- joint j5_tool_roll: origin xyz=0.0285 -0.0487 0.0000 -> xyz=0.0380 0.0420 0.0000

Commit message: Mate-composed assembly + correct face-to-face drive mating
Rebuild arm_assembly by MATING parts from the vendor geometry instead of typed
joint origins: each part exposes mate_frames() (PROX/DIST connectors), the chain
composes them, and the URDF joint origins/axes + the CAD preview are all derived
from the same mated Locations (verified rpy round-trips exactly).

Fix the drive mate to match the real hardware (per a photo of the build): a
drive joins FACE-TO-FACE -- the mount-plate boss-base face (z=6, where the bearing
boss rises) seats against the body's OPEN bore face, the boss dropping into the
bore so the body spins on it. The body mate Z points OUT of the open face so it
receives the boss (earlier it gapped/interfered).

Rest-pose clocking (arm straight up) still WIP; mating geometry is correct.

Co-Authored-By: Claude Opus 4.8 <noreply@anthropic.com>

File: sim/arm_trunk.urdf (robot description, URDF)
Before this commit: robot micro_arm, 7 links, 6 joints
Joints:
- joint j1_yaw: axis 0 0 1 -> 0.0 -0.0 -1.0; origin xyz=0.0000 0.0000 0.0470 -> xyz=0.00000 0.00000 0.00600 rpy=-3.14159 -0.00000 0.00000
- joint j2_shoulder: axis 0 1 0 -> 0.0 1.0 -0.0; origin xyz=0.0000 0.0360 0.0420 -> xyz=0.02590 0.00000 0.04220 rpy=-3.14159 0.00000 1.57080
- joint j3_elbow: axis 0 1 0 -> 0.0 1.0 -0.0; origin xyz=0.0750 -0.0046 0.0000 -> xyz=0.07500 -0.01220 0.00000 rpy=-3.14159 0.00000 -3.14159
- joint j4_wrist_pitch: axis 0 1 0 -> 0.0 -0.0 -1.0; origin xyz=0.0520 -0.0046 0.0000 -> xyz=0.05200 -0.00310 -0.00000 rpy=1.57080 -0.00000 0.00000
- joint j5_tool_roll: axis 1 0 0 -> 1.0 0.0 0.0; origin xyz=0.0380 0.0420 0.0000 -> xyz=0.03500 0.00000 0.04220 rpy=0.00000 1.57080 0.00000

Commit message: Revert assembly to hand-placed version (the mate-composed one was worse)
The mate-composition rewrite collapsed/interfered; roll arm_assembly + URDF back
to 4e20e66 which reads as the arm (base->shoulder->elbow->wrist->gripper). The
parts' mate_frames() stay (harmless, unused) as foundation if revisited. Next:
fix the remaining joint mating gaps surgically against the build photo.

Co-Authored-By: Claude Opus 4.8 <noreply@anthropic.com>

File: sim/arm_trunk.urdf (robot description, URDF)
Before this commit: robot micro_arm, 7 links, 6 joints
Joints:
- joint j1_yaw: axis 0.0 -0.0 -1.0 -> 0 0 1; origin xyz=0.00000 0.00000 0.00600 rpy=-3.14159 -0.00000 0.00000 -> xyz=0.0000 0.0000 0.0470
- joint j2_shoulder: axis 0.0 1.0 -0.0 -> 0 1 0; origin xyz=0.02590 0.00000 0.04220 rpy=-3.14159 0.00000 1.57080 -> xyz=0.0000 0.0360 0.0420
- joint j3_elbow: axis 0.0 1.0 -0.0 -> 0 1 0; origin xyz=0.07500 -0.01220 0.00000 rpy=-3.14159 0.00000 -3.14159 -> xyz=0.0750 -0.0046 0.0000
- joint j4_wrist_pitch: axis 0.0 -0.0 -1.0 -> 0 1 0; origin xyz=0.05200 -0.00310 -0.00000 rpy=1.57080 -0.00000 0.00000 -> xyz=0.0520 -0.0046 0.0000
- joint j5_tool_roll: axis 1.0 0.0 0.0 -> 1 0 0; origin xyz=0.03500 0.00000 0.04220 rpy=0.00000 1.57080 0.00000 -> xyz=0.0380 0.0420 0.0000
